Commit message: First Navigation

File: src/aic26_description/urdf/gazebo_camera.xacro (robot description, xacro)
@@ -1,61 +1,62 @@
+<?xml version="1.0"?>
 <robot name="camera" xmlns:xacro="http://wiki.ros.org/xacro">
-    <xacro:property name="mount_length" value="0.005" />
-    <xacro:property name="mount_width" value="0.008" />
-    <xacro:property name="mount_height" value="${support_length * 2 / 3}" />
-    <xacro:property name="mount_x" value="0.08" />
-    <xacro:property name="mount_y" value="0.0" />
-    <xacro:property name="mount_z" value="${base_link_height / 2 + support_length / 3}" />
-    <xacro:property name="mount_m" value="0.002" />
+    <xacro:property name="mount_length" value="0.005"/>
+    <xacro:property name="mount_width" value="0.008"/>
+    <xacro:property name="mount_height" value="${support_length * 2 / 3}"/>
+    <xacro:property name="mount_x" value="0.08"/>
+    <xacro:property name="mount_y" value="0.0"/>
+    <xacro:property name="mount_z" value="${base_link_height / 2 + support_length / 3}"/>
+    <xacro:property name="mount_m" value="0.002"/>
     <link name="mount">
         <visual>
             <geometry>
-                <box size="${mount_length} ${mount_width} ${mount_height}" rpy="0 0 0" />
+                <box size="${mount_length} ${mount_width} ${mount_height}"/>
             </geometry>
-            <origin size="0.0 0.0 0.0" rpy="0.0 0.0 0.0" />
-            <material name="black" />
+            <origin xyz="0.0 0.0 0.0" rpy="0.0 0.0 0.0"/>
+            <material name="black"/>
         </visual>
         <collision>
             <geometry>
-                <box size="${mount_length} ${mount_width} ${mount_height}" rpy="0 0 0" />
+                <box size="${mount_length} ${mount_width} ${mount_height}"/>
             </geometry>
-            <origin size="0.0 0.0 0.0" rpy="0.0 0.0 0.0" />
+            <origin xyz="0.0 0.0 0.0" rpy="0.0 0.0 0.0"/>
         </collision>
-        <xacro:Box_inertial_matrix m="${mount_m}" l="${mount_length}" w="${mount_width}" h="${mount_height}" />
+        <xacro:Box_inertial_matrix m="${mount_m}" l="${mount_length}" w="${mount_width}" h="${mount_height}"/>
     </link>
     <joint name="mount2base_link" type="fixed">
-        <parent link="base_link" />
-        <child link="mount" />
-        <origin xyz="${mount_x} ${mount_y} ${mount_z}" />
+        <parent link="base_link"/>
+        <child link="mount"/>
+        <origin xyz="${mount_x} ${mount_y} ${mount_z}"/>
     </joint>
     <gazebo reference="mount">
         <material>Gazebo/FlatBlack</material>
     </gazebo>
-    <xacro:property name="camera_length" value="0.01" />
-    <xacro:property name="camera_width" value="0.03" />
-    <xacro:property name="camera_height" value="0.02" />
-    <xacro:property name="camera_x" value="${mount_x + mount_length / 2 + camera_length / 2}" />
-    <xacro:property name="camera_y" value="0.0" />
-    <xacro:property name="camera_z" value="${mount_z + mount_height / 4}" />
-    <xacro:property name="camera_m" value="0.01" />
+    <xacro:property name="camera_length" value="0.01"/>
+    <xacro:property name="camera_width" value="0.03"/>
+    <xacro:property name="camera_height" value="0.02"/>
+    <xacro:property name="camera_x" value="${mount_x + mount_length / 2 + camera_length / 2}"/>
+    <xacro:property name="camera_y" value="0.0"/>
+    <xacro:property name="camera_z" value="${mount_z + mount_height / 4}"/>
+    <xacro:property name="camera_m" value="0.01"/>
     <link name="camera">
         <visual>
             <geometry>
-                <box size="${camera_length} ${camera_width} ${camera_height}" />
+                <box size="${camera_length} ${camera_width} ${camera_height}"/>
             </geometry>
-            <origin xyz="0.0 0.0 0.0" rpy="0.0 0.0 0.0" />
-            <material name="black" />
+            <origin xyz="0.0 0.0 0.0" rpy="0.0 0.0 0.0"/>
+            <material name="black"/>
         </visual>
         <collision>
             <geometry>
-                <box size="${camera_length} ${camera_width} ${camera_height}" />
+                <box size="${camera_length} ${camera_width} ${camera_height}"/>
             </geometry>
-            <origin xyz="0.0 0.0 0.0" rpy="0.0 0.0 0.0" />
+            <origin xyz="0.0 0.0 0.0" rpy="0.0 0.0 0.0"/>
         </collision>
-        <xacro:Box_inertial_matrix m="${camera_m}" l="${camera_length}" w="${camera_width}" h="${camera_height}" />
+        <xacro:Box_inertial_matrix m="${camera_m}" l="${camera_length}" w="${camera_width}" h="${camera_height}"/>
     </link>
     <joint name="camera2mount" type="fixed">
-        <parent link="base_link" />
-        <child link="camera" />
-        <origin xyz="${camera_x} ${camera_y} ${camera_z}" />
+        <parent link="mount"/>
+        <child link="camera"/>
+        <origin xyz="${camera_x} ${camera_y} ${camera_z}"/>
     </joint>
     <gazebo reference="camera">

File: src/aic26_description/urdf/gazebo_head.xacro (robot description, xacro)
@@ -1,2 +1,3 @@
+<?xml version="1.0"?>
 <robot name="base" xmlns:xacro="http://wiki.ros.org/xacro">
     <xacro:macro name="sphere_inertial_matrix" params="m r">

File: src/aic26_description/urdf/gazebo_laser.xacro (robot description, xacro)
@@ -1,2 +1,3 @@
+<?xml version="1.0"?>
 <robot name="my_laser" xmlns:xacro="http://wiki.ros.org/xacro">
     <xacro:property name="support_length" value="0.04" />

Commit message: Fine Decision

File: src/aic26_description/urdf/gazebo_camera.xacro (robot description, xacro)
@@ -4,5 +4,5 @@
     <xacro:property name="mount_width" value="0.008"/>
     <xacro:property name="mount_height" value="${support_length * 2 / 3}"/>
-    <xacro:property name="mount_x" value="0.08"/>
+    <xacro:property name="mount_x" value="0.10"/>
     <xacro:property name="mount_y" value="0.0"/>
     <xacro:property name="mount_z" value="${base_link_height / 2 + support_length / 3}"/>
@@ -65,5 +65,5 @@
         <update_rate>30.0</update_rate>
         <camera name="head">
-            <horizontal_fov>1.570796</horizontal_fov>
+            <horizontal_fov>1.745329</horizontal_fov>
             <image>
                 <width>1280</width>

Commit message: Fine Decision

File: src/aic26_description/urdf/gazebo_camera.xacro (robot description, xacro)
@@ -4,5 +4,5 @@
     <xacro:property name="mount_width" value="0.008"/>
     <xacro:property name="mount_height" value="${support_length * 2 / 3}"/>
-    <xacro:property name="mount_x" value="0.10"/>
+    <xacro:property name="mount_x" value="0.09"/>
     <xacro:property name="mount_y" value="0.0"/>
     <xacro:property name="mount_z" value="${base_link_height / 2 + support_length / 3}"/>
@@ -65,5 +65,5 @@
         <update_rate>30.0</update_rate>
         <camera name="head">
-            <horizontal_fov>1.745329</horizontal_fov>
+            <horizontal_fov>1.570796</horizontal_fov>
             <image>
                 <width>1280</width>

Commit message: Gazebo Plus

File: src/aic26_description/urdf/gazebo_camera.xacro (robot description, xacro)
@@ -35,7 +35,7 @@
     <xacro:property name="camera_width" value="0.03"/>
     <xacro:property name="camera_height" value="0.02"/>
-    <xacro:property name="camera_x" value="${mount_x + mount_length / 2 + camera_length / 2}"/>
+    <xacro:property name="camera_x" value="${mount_length / 2 + camera_length / 2}"/>
     <xacro:property name="camera_y" value="0.0"/>
-    <xacro:property name="camera_z" value="${mount_z + mount_height / 4}"/>
+    <xacro:property name="camera_z" value="${mount_height / 4}"/>
     <xacro:property name="camera_m" value="0.01"/>
     <link name="camera">

Commit message: Format Revise

File: src/aic26_description/urdf/gazebo_camera.xacro (robot description, xacro)
@@ -63,36 +63,36 @@
         <material>Gazebo/Indigo</material>
         <sensor type="camera" name="camera_node">
-        <update_rate>30.0</update_rate>
-        <camera name="head">
-            <horizontal_fov>1.570796</horizontal_fov>
-            <image>
-                <width>1280</width>
-                <height>720</height>
-                <format>R8G8B8</format>
-            </image>
-            <clip>
-                <near>0.02</near>
-                <far>300</far>
-            </clip>
-            <noise>
-                <type>gaussian</type>
-                <mean>0.0</mean>
-                <stddev>0.007</stddev>
-            </noise>
-        </camera>
-        <plugin name="gazebo_camera" filename="libgazebo_ros_camera.so">
-            <alwaysOn>true</alwaysOn>
-            <updateRate>0.0</updateRate>
-            <cameraName>camera</cameraName>
-            <imageTopicName>image_raw</imageTopicName>
-            <cameraInfoTopicName>camera_info</cameraInfoTopicName>
-            <frameName>camera</frameName>
-            <hackBaseline>0.07</hackBaseline>
-            <distortionK1>0.0</distortionK1>
-            <distortionK2>0.0</distortionK2>
-            <distortionK3>0.0</distortionK3>
-            <distortionT1>0.0</distortionT1>
-            <distortionT2>0.0</distortionT2>
-        </plugin>
+            <update_rate>30.0</update_rate>
+            <camera name="head">
+                <horizontal_fov>1.570796</horizontal_fov>
+                <image>
+                    <width>1280</width>
+                    <height>720</height>
+                    <format>R8G8B8</format>
+                </image>
+                <clip>
+                    <near>0.02</near>
+                    <far>300</far>
+                </clip>
+                <noise>
+                    <type>gaussian</type>
+                    <mean>0.0</mean>
+                    <stddev>0.007</stddev>
+                </noise>
+            </camera>
+            <plugin name="gazebo_camera" filename="libgazebo_ros_camera.so">
+                <alwaysOn>true</alwaysOn>
+                <updateRate>0.0</updateRate>
+                <cameraName>camera</cameraName>
+                <imageTopicName>image_raw</imageTopicName>
+                <cameraInfoTopicName>camera_info</cameraInfoTopicName>
+                <frameName>camera</frameName>
+                <hackBaseline>0.07</hackBaseline>
+                <distortionK1>0.0</distortionK1>
+                <distortionK2>0.0</distortionK2>
+                <distortionK3>0.0</distortionK3>
+                <distortionT1>0.0</distortionT1>
+                <distortionT2>0.0</distortionT2>
+            </plugin>
         </sensor>
     </gazebo>

File: src/aic26_description/urdf/gazebo_car_union.xacro (robot description, xacro)
@@ -6,5 +6,6 @@
   <xacro:include filename="gazebo_camera.xacro"/>
   <xacro:include filename="gazebo_light.xacro"/>
-  <!-- Keep the existing navigation API while using the VM project's four-wheel skid drive. -->
+  <!-- Keep the /cmd_vel and /odom interface while using a four-wheel
+       skid-steer drive. -->
   <gazebo>
     <plugin name="mobile_base_controller" filename="libgazebo_ros_skid_steer_drive.so">

File: src/aic26_description/urdf/gazebo_head.xacro (robot description, xacro)
@@ -12,16 +12,16 @@
         <inertial>
             <mass value="${m}" />
-            <inertia ixx="${m*(3*r*r+h*h)/12}" ixy = "0" ixz = "0"
-                iyy="${m*(3*r*r+h*h)/12}" iyz = "0"
+            <inertia ixx="${m*(3*r*r+h*h)/12}" ixy="0" ixz="0"
+                iyy="${m*(3*r*r+h*h)/12}" iyz="0"
                 izz="${m*r*r/2}" />
         </inertial>
     </xacro:macro>
     <xacro:macro name="Box_inertial_matrix" params="m l w h">
-       <inertial>
-               <mass value="${m}" />
-               <inertia ixx="${m*(h*h + l*l)/12}" ixy = "0" ixz = "0"
-                   iyy="${m*(w*w + l*l)/12}" iyz= "0"
-                   izz="${m*(w*w + h*h)/12}" />
-       </inertial>
-   </xacro:macro>
+        <inertial>
+            <mass value="${m}" />
+            <inertia ixx="${m*(h*h + l*l)/12}" ixy="0" ixz="0"
+                iyy="${m*(w*w + l*l)/12}" iyz="0"
+                izz="${m*(w*w + h*h)/12}" />
+        </inertial>
+    </xacro:macro>
 </robot>

File: src/aic26_description/urdf/gazebo_light.xacro (robot description, xacro)
@@ -1,4 +1,4 @@
 <?xml version="1.0"?>
-<robot xmlns:xacro="http://www.ros.org/wiki/xacro">
+<robot xmlns:xacro="http://wiki.ros.org/xacro">
   <xacro:property name="light_length" value="0.006" />
   <xacro:property name="light_radius" value="0.015" />
